Commit message: Mass and inertia added

File: urdf/xr1urdf.urdf (robot description, URDF)
Before this commit: robot xr1urdf, 51 links, 50 joints
Links:
- link Back_Link: mass 0.704367292272377 -> 13.87
- link Head_Link: mass 0.0888013589166292 -> 1.661
- link Knee_Link: mass 0.0222634661487604 -> 8.175
- link Left_1_1_Link: mass 0.00270491937647517 -> 0.06844
- link Left_1_2_Link: mass 0.00170025166301577 -> 0.01812
- link Left_2_1_Link: mass 0.00257050995799412 -> 0.05105
- link Left_2_2_Link: mass 0.00174377331167473 -> 0.01234
- link Left_2_3_Link: mass 0.0017150608380904 -> 0.006588
- link Left_3_1_Link: mass 0.00266106740478141 -> 0.05197
- link Left_3_2_Link: mass 0.00174377422788023 -> 0.01299
- link Left_3_3_Link: mass 0.00171505840101367 -> 0.006329
- link Left_4_1_Link: mass 0.00256743782510478 -> 0.04255
- link Left_4_2_Link: mass 0.00174377568021046 -> 0.01146
- link Left_4_3_Link: mass 0.00171506109632343 -> 0.00662
- link Left_5_1_Link: mass 0.00247216445342281 -> 0.0465
- link Left_5_2_Link: mass 0.00174377457432162 -> 0.01531
- link Left_5_3_Link: mass 0.00171506218865776 -> 0.007844
- link Left_Arm_Link: mass 0.0603362552750754 -> 1.022
- link Left_Elbow_Link: mass 0.00808614997974233 -> 0.7854
- link Left_Forearm_Link: mass 0.14751742316436 -> 0.6233
- link Left_Hand_Link: mass 0.0154024949242438 -> 0.1449
- link Left_Shoulder_Link: mass 0.0156440867968973 -> 0.8107
- link Left_Wrist_Link: mass 0.0646072856279338 -> 0.5487
- link Left_Wrist_Link2: mass 0.0361826967926398 -> 0.5362
- link Leg_Link: mass 0.322927964021912 -> 0.32293
- link Neck_Link: mass 0.0103446909694818 -> 0.6805
- link Neck_Link2: mass 0.0140062146286296 -> 0.4417
- link Right_1_1_Link: mass 0.0027049193764752 -> 0.0648
- link Right_1_2_Link: mass 0.00170025166301581 -> 0.01812
- link Right_2_1_Link: mass 0.00257050995799409 -> 0.05105
- link Right_2_2_Link: mass 0.00174377331167817 -> 0.01234
- link Right_2_3_Link: mass 0.0017150608380904 -> 0.006588
- link Right_3_1_Link: mass 0.00266106740478136 -> 0.05197
- link Right_3_2_Link: mass 0.00174377422787818 -> 0.01299
- link Right_3_3_Link: mass 0.00171505840101365 -> 0.006329
- link Right_4_1_Link: mass 0.00256743782510473 -> 0.04255
- link Right_4_2_Link: mass 0.00174377568020993 -> 0.01146
- link Right_4_3_Link: mass 0.00171506109632349 -> 0.00662
- link Right_5_1_Link: mass 0.00247216445342274 -> 0.0465
- link Right_5_2_Link: mass 0.0017437745743221 -> 0.01531
- link Right_5_3_Link: mass 0.00171506218865772 -> 0.007844
- link Right_Arm_Link: mass 0.0603362552750853 -> 1.022
- link Right_Elbow_Link: mass 0.00808614997974196 -> 0.7854
- link Right_Foream_Link: mass 0.14751742316687 -> 0.6233
- link Right_Hand_Link: mass 0.0154024961513519 -> 0.1449
- link Right_Shoulder_Link: mass 0.0156440867968964 -> 0.8107
- link Right_Wrist_Link: mass 0.0646072856279335 -> 0.5484
- link Right_Wrist_Link2: mass 0.0361826967926398 -> 0.5362
- link Thigh_Link: mass 5.12610482593271 -> 0.8847
- link Thigh_Link2: mass 5.12610482593271 -> 0.6035
- link base_link: mass 3.70172320150886 -> 36.19
Joints:
- joint Back_X: origin xyz=-0.0136036359907622 -5.7629583447044E-05 0.424066015793186 rpy=-1.57066035921997 -0.0320680548961984 -4.35946841023116E-06 -> xyz=-0.013604 -5.763E-05 0.42407 rpy=-1.5707 -0.032068 -4.3595E-06
- joint Back_Y: origin xyz=-0.0138647143421331 -0.105654674591013 -2.69257267197509E-05 rpy=-1.5707963267949 0 -1.57124614957808 -> xyz=-0.013865 -0.10565 -2.6926E-05 rpy=-1.5708 0 -1.5712
- joint Back_Z: axis -0.0325121474774201 -0.000135825825076976 0.999471331163506 -> -0.032512 -0.00013583 0.99947; origin xyz=0 0 0 rpy=1.57066042912579 0 -0.00121611800675794 -> xyz=0 0 0 rpy=1.5707 0 -0.0012161
- joint Knee_X: origin xyz=5.49383760162785E-05 -0.0131434525992938 0.404049107981184 rpy=-1.5707963267949 0.0337339959823619 -1.5707963267949 -> xyz=5.4938E-05 -0.013143 0.40405 rpy=-1.5708 0.033734 -1.5708
- joint Left_Elbow_Z: origin xyz=0 0.0513427925767579 0.00307040580185031 rpy=-1.5707963267949 0 1.5707963267949 -> xyz=0 0.051343 0.0030704 rpy=-1.5708 0 1.5708
- joint Left_Shoulder_X: origin xyz=0.258474937704725 -0.151060434921511 0.00158495021114652 rpy=1.5707963267949 -1.5707963267949 0 -> xyz=0.25847 -0.15106 0.001585 rpy=1.5708 -1.5708 0
- joint Left_Shoulder_Y: origin xyz=0 0 0 rpy=1.5707963267949 0 1.5707963267949 -> xyz=0 0 0 rpy=1.5708 0 1.5708
- joint Leg_D: origin xyz=0 0 0 rpy=0 0 6.93889390390723E-18 -> xyz=0 0 0 rpy=0 0 6.9389E-18
- joint Right_Elbow_Z: origin xyz=-0.000167064372992076 -0.0516466951322389 0.0029862446509249 rpy=-1.61480130234895 0 1.57010549404216 -> xyz=-0.00016706 -0.051647 0.0029862 rpy=-1.6148 0 1.5701
- joint Right_Shoulder_Y: axis -0.0439907642815591 3.03902656184142E-05 0.999031937294477 -> -0.043991 3.039E-05 0.99903; origin xyz=0 0 0 rpy=1.57082668764085 -1.33689101189151E-06 1.61480129184152 -> xyz=0 0 0 rpy=1.5708 -1.3369E-06 1.6148

Commit message: Left Wrist Fixed

File: urdf/xr1urdf.urdf (robot description, URDF)
Before this commit: robot xr1urdf, 51 links, 50 joints
Joints:
- removed joint Right_3_1_Link
- added joint Right_3_1_Joint: type continuous, parent Right_Hand_Link, child Right_3_1_Link, origin xyz=0.0764901009021922 -0.00561489331473879 -0.00175480169051168 rpy=1.5707963267949 -1.5707963267949 0, axis 0 0 1
- joint Left_1_1_Joint: origin xyz=0.0434901201851731 0.0577281894210584 -0.0144771062637427 rpy=0 -1.00156316575 1.94835151482426 -> xyz=0.0463873711048263 -0.0227514450525238 -0.0270481463075324 rpy=0 -1.00156316575 1.94835151482426
- joint Left_2_1_Joint: origin xyz=0.0713207399971868 0.0593046011451485 0.0116439951156551 rpy=1.5707963267949 -1.5707963267949 0 -> xyz=0.07421799091684 -0.0211750333284337 -0.000927044928134585 rpy=1.5707963267949 -1.5707963267949 0
- joint Left_3_1_Joint: origin xyz=0.073592849982539 0.0748647411588435 0.0143258417343013 rpy=1.5707963267949 -1.5707963267949 0 -> xyz=0.0764901009021922 -0.00561489331473879 0.00175480169051168 rpy=1.5707963267949 -1.5707963267949 0
- joint Left_4_1_Joint: origin xyz=0.0706317293770647 0.0901645061794522 0.0135342539047116 rpy=1.5707963267949 -1.5707963267949 0 -> xyz=0.073528980296718 0.00968487170586999 0.000963213860921908 rpy=1.5707963267949 -1.5707963267949 0
- joint Left_5_1_Joint: origin xyz=0.0673939669258992 0.105356641006828 0.0129590738510026 rpy=1.5707963267949 -1.5707963267949 0 -> xyz=0.0702912178455524 0.0248770065332455 0.00038803380721289 rpy=1.5707963267949 -1.5707963267949 0
- joint Left_Wrist_Y: origin xyz=0.0883192894929252 0.0118949477766215 0.222176978855445 rpy=-1.5707963267949 0 -1.5707963267949 -> xyz=0.00784287714185615 0.000519681604099265 0.219279727935792 rpy=-1.5707963267949 0 -1.5707963267949

Commit message: Joint Limit Added

File: urdf/xr1urdf.urdf (robot description, URDF)
Before this commit: robot xr1urdf, 51 links, 50 joints
Joints:
- removed joint Left_4_3_Link
- added joint Left_4_3_Joint: type revolute, parent Left_4_2_Link, child Left_4_3_Link, origin xyz=0 -0.0220256805419927 0 rpy=0 0 0, axis 0 0 -1, limit lower=0.0 upper=1.74 effort=30 velocity=3.14
- joint Back_X: limit (none) -> lower=-0.691 upper=0.691 effort=30 velocity=3.14; type continuous -> revolute
- joint Back_Y: limit (none) -> lower=-1.01 upper=1.01 effort=30 velocity=3.14; type continuous -> revolute
- joint Back_Z: limit (none) -> lower=-1.57 upper=1.57 effort=30 velocity=3.14; type continuous -> revolute
- joint Head_Y: limit (none) -> lower=-1.26 upper=1.26 effort=30 velocity=3.14; type continuous -> revolute
- joint Knee_X: limit (none) -> lower=-0.691 upper=0.691 effort=30 velocity=3.14; type continuous -> revolute
- joint Left_1_1_Joint: limit (none) -> lower=0.0 upper=1.21 effort=30 velocity=3.14; type continuous -> revolute
- joint Left_1_2_Joint: limit (none) -> lower=0.0 upper=1.45 effort=30 velocity=3.14; type continuous -> revolute
- joint Left_2_1_Joint: axis 0 0 1 -> 0 0 -1; limit (none) -> lower=0.0 upper=1.00 effort=30 velocity=3.14; type continuous -> revolute
- joint Left_2_2_Joint: axis 0 0 1 -> 0 0 -1; limit (none) -> lower=0.0 upper=1.20 effort=30 velocity=3.14; type continuous -> revolute
- joint Left_2_3_Joint: axis 0 0 1 -> 0 0 -1; limit (none) -> lower=0.0 upper=1.45 effort=30 velocity=3.14; type continuous -> revolute
- joint Left_3_1_Joint: axis 0 0 1 -> 0 0 -1; limit (none) -> lower=0.0 upper=1.17 effort=30 velocity=3.14; type continuous -> revolute
- joint Left_3_2_Joint: axis 0 0 1 -> 0 0 -1; limit (none) -> lower=0.0 upper=1.41 effort=30 velocity=3.14; type continuous -> revolute
- joint Left_3_3_Joint: axis 0 0 1 -> 0 0 -1; limit (none) -> lower=0.0 upper=1.69 effort=30 velocity=3.14; type continuous -> revolute
- joint Left_4_1_Joint: axis 0 0 1 -> 0 0 -1; limit (none) -> lower=0.0 upper=1.20 effort=30 velocity=3.14; type continuous -> revolute
- joint Left_4_2_Joint: axis 0 0 1 -> 0 0 -1; limit (none) -> lower=0.0 upper=1.45 effort=30 velocity=3.14; type continuous -> revolute
- joint Left_5_1_Joint: axis 0 0 1 -> 0 0 -1; limit (none) -> lower=0.0 upper=1.30 effort=30 velocity=3.14; type continuous -> revolute
- joint Left_5_2_Joint: axis 0 0 1 -> 0 0 -1; limit (none) -> lower=0.0 upper=1.56 effort=30 velocity=3.14; type continuous -> revolute
- joint Left_5_3_Joint: axis 0 0 1 -> 0 0 -1; limit (none) -> lower=0.0 upper=1.87 effort=30 velocity=3.14; type continuous -> revolute
- joint Left_Elbow_X: limit (none) -> lower=-1.57 upper=0.1 effort=30 velocity=3.14; type continuous -> revolute
- joint Left_Elbow_Z: limit (none) -> lower=-3.14 upper=3.14 effort=30 velocity=3.14; type continuous -> revolute
- joint Left_Shoulder_X: limit (none) -> lower=-2.26 upper=2.26 effort=30 velocity=3.14; type continuous -> revolute
- joint Left_Shoulder_Y: limit (none) -> lower=-0.188 upper=1.88 effort=30 velocity=3.14; type continuous -> revolute
- joint Left_Wrist_X: limit (none) -> lower=-0.88 upper=0.754 effort=30 velocity=3.14; type continuous -> revolute
- joint Left_Wrist_Y: limit (none) -> lower=-1.07 upper=1.13 effort=30 velocity=3.14; type continuous -> revolute
- joint Left_Wrist_Z: limit (none) -> lower=-3.14 upper=3.14 effort=30 velocity=3.14; type continuous -> revolute
- joint Neck_X: limit (none) -> lower=-1.01 upper=0.628 effort=30 velocity=3.14; type continuous -> revolute
- joint Neck_Z: limit (none) -> lower=-1.57 upper=1.57 effort=30 velocity=3.14; type continuous -> revolute
- joint Right_1_1_Joint: limit (none) -> lower=0.0 upper=1.21 effort=30 velocity=3.14; type continuous -> revolute
- joint Right_1_2_Joint: limit (none) -> lower=0.0 upper=1.45 effort=30 velocity=3.14; type continuous -> revolute
- joint Right_2_1_Joint: limit (none) -> lower=0.0 upper=1.00 effort=30 velocity=3.14; type continuous -> revolute
- joint Right_2_2_Joint: limit (none) -> lower=0.0 upper=1.20 effort=30 velocity=3.14; type continuous -> revolute
- joint Right_2_3_Joint: limit (none) -> lower=0.0 upper=1.45 effort=30 velocity=3.14; type continuous -> revolute
- joint Right_3_1_Joint: limit (none) -> lower=0.0 upper=1.17 effort=30 velocity=3.14; type continuous -> revolute
- joint Right_3_2_Joint: limit (none) -> lower=0.0 upper=1.41 effort=30 velocity=3.14; type continuous -> revolute
- joint Right_3_3_Joint: limit (none) -> lower=0.0 upper=1.69 effort=30 velocity=3.14; type continuous -> revolute
- joint Right_4_1_Joint: limit (none) -> lower=0.0 upper=1.20 effort=30 velocity=3.14; type continuous -> revolute
- joint Right_4_2_Joint: limit (none) -> lower=0.0 upper=1.45 effort=30 velocity=3.14; type continuous -> revolute
- joint Right_4_3_Joint: limit (none) -> lower=0.0 upper=1.74 effort=30 velocity=3.14; type continuous -> revolute
- joint Right_5_1_Joint: limit (none) -> lower=0.0 upper=1.30 effort=30 velocity=3.14; type continuous -> revolute
- joint Right_5_2_Joint: limit (none) -> lower=0.0 upper=1.56 effort=30 velocity=3.14; type continuous -> revolute
- joint Right_5_3_Joint: limit (none) -> lower=0.0 upper=1.87 effort=30 velocity=3.14; type continuous -> revolute
- joint Right_Elbow_X: limit (none) -> lower=-1.57 upper=0.1 effort=30 velocity=3.14; type continuous -> revolute
- joint Right_Elbow_Z: limit (none) -> lower=-3.14 upper=3.14 effort=30 velocity=3.14; type continuous -> revolute
- joint Right_Shoulder_X: limit (none) -> lower=-2.26 upper=2.26 effort=30 velocity=3.14; type continuous -> revolute
- joint Right_Shoulder_Y: limit (none) -> lower=-1.88 upper=0.188 effort=30 velocity=3.14; type continuous -> revolute
- joint Right_Wrist_X: limit (none) -> lower=-0.88 upper=0.754 effort=30 velocity=3.14; type continuous -> revolute
- joint Right_Wrist_Y: limit (none) -> lower=-1.13 upper=1.07 effort=30 velocity=3.14; type continuous -> revolute
- joint Right_Wrist_Z: limit (none) -> lower=-3.14 upper=3.14 effort=30 velocity=3.14; type continuous -> revolute
